Commit message: Retirei a camara e adicionei o aruco

File: ur_e_description/urdf/common.gazebo.xacro (robot description, xacro)
@@ -20,4 +20,19 @@
     </plugin>
 -->
+	<plugin name="gazebo_grasp_fix" filename="/home/nacl/catkin_ws/devel/lib/libgazebo_grasp_fix.so">
+		<arm>
+			<arm_name>ur10eRobot</arm_name>
+			<palm_link>wrist_3_link</palm_link>
+			<gripper_link>left_finger_link</gripper_link>
+			<gripper_link>right_finger_link</gripper_link>
+		</arm>
+		<forces_angle_tolerance>100</forces_angle_tolerance>
+		<update_rate>50</update_rate>
+		<grip_count_threshold>4</grip_count_threshold>
+		<max_grip_count>8</max_grip_count>
+		<release_tolerance>0.002</release_tolerance>
+		<disable_collisions_on_attach>false</disable_collisions_on_attach>
+		<contact_topic>__default_topic__</contact_topic>
+	</plugin>
   </gazebo>
 </robot>

File: ur_e_description/urdf/ur.gazebo.xacro (robot description, xacro)
@@ -34,5 +34,5 @@
   </xacro:macro>
   <xacro:macro name="sim_3dsensor" params="prefix">
-      <gazebo reference="${prefix}_rgb_frame">
+      <gazebo reference="${prefix}_depth_frame">
           <sensor type="depth" name="camera">
               <always_on>true</always_on>

File: ur_e_description/urdf/ur10e_joint_limited_robot.urdf.xacro (robot description, xacro)
@@ -16,9 +16,15 @@
 />
   <!-- sensor -->
-  <xacro:include filename="$(find ur_e_description)/urdf/astra.urdf.xacro" />
-  <xacro:sensor_astra parent="ee_link" prefix="camera">
-      <origin xyz="0.041311319304504816 -0.06402544453787727 0.044527571211305426"
-              rpy="3.13766148064 -0.00787797070144 0.000110993634886"/>
-  </xacro:sensor_astra>
+  <!--xacro:include filename="$(find ur_e_description)/urdf/astra.urdf.xacro" />
+  <xacro:sensor_astra parent="world" prefix="camera">
+      <origin xyz="1.2 0 1" rpy="${0} ${pi - 2*pi/5} ${0}"/>			<!- - Vista normal - ->
+      <!- -origin xyz="1 0.6 1" rpy="${0} ${pi - 2*pi/5} ${pi/2}"/- -> 	<!- - Vista lateral - ->
+	  <!- -origin xyz="1.2 0 1" rpy="${0} ${pi - 3*pi/5} ${pi}"/- ->		<!- - Vista invertida - ->
+	  <!- -origin xyz="0.92 0.1 1" rpy="${0} ${pi/2} ${0}"/- ->					<!- - Vista diretamente de cima - ->
+  </xacro:sensor_astra-->
+  <xacro:include filename="$(find ur_e_description)/urdf/aruco/aruco_582.urdf.xacro" />
+  <xacro:aruco parent="ee_link" prefix="aruco">
+  	<origin xyz="0.032 0 -0.034" rpy="${0} ${0} ${0}"/>
+</xacro:aruco>
   <link name="world" />
   <joint name="world_joint" type="fixed">
